File: MD2.sch (KiCad schematic (older format))
At the start: 41 parts, among them IC4 A3921KLPTR-T, IC5 SI4900DY-T1-E3, IC6 SI4900DY-T1-E3, J4 Connector_Generic_Conn_01x05, J5 Connector_Generic_Conn_01x02, J6 Connector_Generic_Conn_01x02, SW2 SW_Push, U5 FODM217A, U6 FODM217A, U7 FODM217A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

Commit message: シンボルの挿入まで完成
Parts:
- removed C11: 220u, Capacitor_SMD:CP_Elec_5x3, symbol Device:CP
- removed SW2: SW_Push, Button_Switch_SMD:SW_SPST_B3U-1000P, symbol Switch:SW_Push
- added SW2: SW_MEC_5G, Button_Switch_SMD:SW_Push_1P1T_NO_CK_KMR2, symbol Switch:SW_MEC_5G
- C12: renamed from C14; value 0.1u -> 1u
- C16: renamed from C18; value 0.22u -> 1u; footprint Capacitor_SMD:C_1206_3216Metric -> Capacitor_SMD:C_0603_1608Metric
- C9: renamed from C10; footprint Capacitor_SMD:CP_Elec_5x3 -> Capacitor_SMD:CP_Elec_10x10
- IC4: symbol SamacSys_Parts:A3921KLPTR-T -> MiniMD-rescue:A3921KLPTR-T-SamacSys_Parts
- IC5, IC6: symbol SamacSys_Parts:SI4900DY-T1-E3 -> MiniMD-rescue:SI4900DY-T1-E3-SamacSys_Parts
- J4: symbol CoulombMini-cache:Connector_Generic_Conn_01x05 -> MiniMD-rescue:Connector_Generic_Conn_01x05-CoulombMini-cache
- J5, J6: symbol CoulombMini-cache:Connector_Generic_Conn_01x02 -> MiniMD-rescue:Connector_Generic_Conn_01x02-CoulombMini-cache
- R30: value 1k -> 100k
- R32: value 1k -> 10k
- renumbered C12 to C10, C13 to C11, C15 to C13, C16 to C14, C17 to C15
Connections:
- net 5V_2: now also C12.1, R31.2; no longer R27.1
- net GND: now also R32.2, SW2.1 (A), SW2.2 (A)
- net VCC: now also R27.1
- net at IC4.24 (RESET), R27.2: now also SW2.3 (B), SW2.4 (B)
- net at IC4.27 (RDEAD): now also R30.1; no longer R32.1
- net at IC4.28 (VDSTH): now also R31.1, R32.1; no longer C12.1
Other:
- moved on the sheet: C12
