File: MiniMD.sch (KiCad schematic (older format))
At the start: 41 parts, among them IC1 A3921KLPTR-T, IC2 SI4900DY-T1-E3, IC3 SI4900DY-T1-E3, J1 Connector_Generic_Conn_01x05, J2 Connector_Generic_Conn_01x02, J3 Connector_Generic_Conn_01x02, SW1 SW_Push, U1 FODM217A, U2 FODM217A, U3 FODM217A, U4 FODM217A

Commit message: シンボルの挿入まで完成
Parts:
- removed C4: 220u, Capacitor_SMD:CP_Elec_5x3, symbol Device:CP
- removed SW1: SW_Push, Button_Switch_SMD:SW_SPST_B3U-1000P, symbol Switch:SW_Push
- added SW1: SW_MEC_5G, Button_Switch_SMD:SW_Push_1P1T_NO_CK_KMR2, symbol Switch:SW_MEC_5G
- C2: value 0.1u -> 1u
- C3: footprint Capacitor_SMD:CP_Elec_5x3 -> Capacitor_SMD:CP_Elec_10x10
- C7: renamed from C8; value 0.22u -> 1u; footprint Capacitor_SMD:C_1206_3216Metric -> Capacitor_SMD:C_0603_1608Metric
- IC1: symbol SamacSys_Parts:A3921KLPTR-T -> MiniMD-rescue:A3921KLPTR-T-SamacSys_Parts
- IC2, IC3: symbol SamacSys_Parts:SI4900DY-T1-E3 -> MiniMD-rescue:SI4900DY-T1-E3-SamacSys_Parts
- J1: symbol CoulombMini-cache:Connector_Generic_Conn_01x05 -> MiniMD-rescue:Connector_Generic_Conn_01x05-CoulombMini-cache
- J2, J3: symbol CoulombMini-cache:Connector_Generic_Conn_01x02 -> MiniMD-rescue:Connector_Generic_Conn_01x02-CoulombMini-cache
- R12: value 1k -> 100k
- R14: value 1k -> 10k
- renumbered C5 to C4, C6 to C5, C7 to C6, C9 to C8
Connections:
- wire segments 179 -> 174

Commit message: 完成
Parts:
- removed J1: Connector_Generic_Conn_01x05, Connector_JST:JST_XH_B5B-XH-A_1x05_P2.50mm_Vertical, symbol MiniMD-rescue:Connector_Generic_Conn_01x05-CoulombMini-cache
- removed R2, R4: 1k, Resistor_SMD:R_0603_1608Metric, symbol Device:R
- removed U2, U4: FODM217A, Package_SO:SOP-4_4.4x2.6mm_P1.27mm, symbol Isolator:FODM217A
- added J2: Conn_01x03, Connector_JST:JST_XH_B3B-XH-A_1x03_P2.50mm_Vertical, symbol Connector_Generic:Conn_01x03
- C5, C6: value 0.22u -> 0.47u
- renumbered C3 to C1, C4 to C2, C8 to C3, C1 to C4, C2 to C8, D3 to D1, D1 to D2, D2 to D3, IC2 to IC1, IC3 to IC2, IC1 to IC3, J2 to J1, R9 to R1, R7 to R10, R18 to R11, R10 to R12, R11 to R13, R12 to R14, R13 to R15, R14 to R16, R6 to R2, R8 to R3, R1 to R4, R15 to R5, R16 to R6, R3 to R7, R17 to R8, R5 to R9, U3 to U2
Connections:
- net 5V_1: now also R2.1, R3.1
- net GND: no longer R2.2, R3.2
- net GND1: now also J2.1 (Pin_1)
- net at IC3.23 (PWMH): now also R3.2; no longer R3.1
- net at IC3.21 (SR): now also R2.2; no longer R2.1
- net at R7.1: now also J2.2 (Pin_2)
- net at R4.1: now also J2.3 (Pin_3)
- net at C5.2, IC1.3 (S2), IC1.7 (D1)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: now also J3.2 (Pin_2); no longer J3.1 (Pin_1)
- net at C6.2, IC2.1 (S1), IC2.5 (D2)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: now also J3.1 (Pin_1); no longer J3.2 (Pin_2)
Other:
- moved on the sheet: J3, R10, R2, R3, R4, R7, U1, U2
